File: boost.kicad_sch (KiCad schematic)
At the start: 19 parts, among them Q1 BSS138, U5 TPS61379QWRTERQ1

Commit message: Started adding new parts to inventree and re-synchronizing here.
Parts:
- R22: footprint (none) -> Resistor_SMD:R_0402_1005Metric; symbol Device:R_US -> #inventree_kicad:R_80K6_0402_1PCT_0W0625; IPN (none) -> 302-0016; InvenTree (none) -> 36; Part URL (none) -> http://10.0.0.33/web/part/36/
- R23: footprint (none) -> Resistor_SMD:R_0402_1005Metric; symbol Device:R_US -> #inventree_kicad:R_825K_0402_1PCT_0W0625; IPN (none) -> 302-0015; InvenTree (none) -> 35; Part URL (none) -> http://10.0.0.33/web/part/35/
- R39: footprint (none) -> Resistor_SMD:R_0402_1005Metric; symbol Device:R_US -> #inventree_kicad:R_470K_0402_1PCT_0W0625; IPN (none) -> 302-0014; InvenTree (none) -> 34; Part URL (none) -> http://10.0.0.33/web/part/34/
Changed lines of the file:
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@@
 	)
 	(symbol
-		(lib_id "Device:R_US")
+		(lib_id "#inventree_kicad:R_80K6_0402_1PCT_0W0625")
 		(at 203.2 125.73 180)
 		(unit 1)
@@
 			)
 		)
-		(property "Footprint" ""
+		(property "Footprint" "Resistor_SMD:R_0402_1005Metric"
 			(at 202.184 125.476 90)
 			(hide yes)
@@
 			)
 		)
-		(property "Description" "Resistor, US symbol"
+		(property "Description" "80.6 kOhm ±1% 0.063W, 1/16W Chip Resistor 0402 (1005 Metric)"
+			(at 203.2 125.73 0)
+			(hide yes)
+			(show_name no)
+			(do_not_autoplace no)
+			(effects
+				(font
+					(size 1.27 1.27)
+				)
+			)
+		)
+		(property "IPN" "302-0016"
+			(at 203.2 125.73 0)
+			(hide yes)
+			(show_name no)
+			(do_not_autoplace no)
+			(effects
+				(font
+					(size 1.27 1.27)
+				)
+			)
+		)
+		(property "InvenTree" "36"
+			(at 203.2 125.73 0)
+			(hide yes)
+			(show_name no)
+			(do_not_autoplace no)
+			(effects
+				(font
+					(size 1.27 1.27)
+				)
+			)
+		)
+		(property "Part URL" "http://10.0.0.33/web/part/36/"
 			(at 203.2 125.73 0)
 			(hide yes)
@@
 	)
 	(symbol
-		(lib_id "Device:R_US")
+		(lib_id "#inventree_kicad:R_825K_0402_1PCT_0W0625")
 		(at 203.2 105.41 180)
 		(unit 1)
@@
 			)
 		)
-		(property "Footprint" ""
+		(property "Footprint" "Resistor_SMD:R_0402_1005Metric"
 			(at 202.184 105.156 90)
 			(hide yes)
@@
 			)
 		)
-		(property "Description" "Resistor, US symbol"
+		(property "Description" "825 kOhm ±1% 0.063W, 1/16W Chip Resistor 0402 (1005 Metric)"
+			(at 203.2 105.41 0)
+			(hide yes)
+			(show_name no)
+			(do_not_autoplace no)
+			(effects
+				(font
+					(size 1.27 1.27)
+				)
+			)
+		)
+		(property "IPN" "302-0015"
+			(at 203.2 105.41 0)
+			(hide yes)
+			(show_name no)
+			(do_not_autoplace no)
+			(effects
+				(font
+					(size 1.27 1.27)
+				)
+			)
+		)
+		(property "InvenTree" "35"
+			(at 203.2 105.41 0)
+			(hide yes)
+			(show_name no)
+			(do_not_autoplace no)
+			(effects
+				(font
+					(size 1.27 1.27)
+				)
+			)
+		)
+		(property "Part URL" "http://10.0.0.33/web/part/35/"
 			(at 203.2 105.41 0)
 			(hide yes)
@@
 	)
 	(symbol
-		(lib_id "Device:R_US")
+		(lib_id "#inventree_kicad:R_470K_0402_1PCT_0W0625")
 		(at 109.22 82.55 0)
 		(unit 1)
@@
 			)
 		)
-		(property "Footprint" ""
+		(property "Footprint" "Resistor_SMD:R_0402_1005Metric"
 			(at 110.236 82.804 90)
 			(hide yes)
@@
 			)
 		)
-		(property "Description" "Resistor, US symbol"
+		(property "Description" "470 kOhm ±1% 0.063W, 1/16W Chip Resistor 0402 (1005 Metric)"
 			(at 109.22 82.55 0)
 			(hide yes)
+			(show_name no)
+			(do_not_autoplace no)
+			(effects
+				(font
+					(size 1.27 1.27)
+				)
+			)
+		)
+		(property "IPN" "302-0014"
+			(at 109.22 82.55 0)
+			(hide yes)
+			(show_name no)
+			(do_not_autoplace no)
+			(effects
+				(font
+					(size 1.27 1.27)
+				)
+			)
+		)
+		(property "InvenTree" "34"
+			(at 109.22 82.55 0)
+			(hide yes)
+			(show_name no)
+			(do_not_autoplace no)
+			(effects
+				(font
+					(size 1.27 1.27)
+				)
+			)
+		)
+		(property "Part URL" "http://10.0.0.33/web/part/34/"
+			(at 109.22 82.55 0)
+			(hide yes)
