File: headphone_amp.kicad_sch (KiCad schematic)
At the start: 0 parts

Commit message: Started Inventree work.
Changed lines of the file:
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@@
 		)
 	)
-	(label "AUDIO_IN"
+	(label "WD_AUDIO_IN"
 		(at 110.49 121.92 0)
 		(effects
@@
 			(project "headphone_amp"
 				(path "/62ffec33-ae93-49a8-bfe6-566578dd8e82"
-					(page "1")
-				)
-			)
+					(page "9")
+				)
+			)

Commit message: Corrected issues Claude identified, added 'poor man's cab filter' on recovery stage per Ihsan.
Other:
- sheet Audio Input ports: added AUDIO_OUT; removed OUT
Changed lines of the file:
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@@
-			)
-		)
-		(pin "OUT" output
-			(at 102.87 149.86 0)
-			(effects
-				(font
-					(size 1.27 1.27)
-				)
-				(justify right)
 			)
 		)
@@
 			(effects
 				(font
+					(size 1.27 1.27)
+				)
+				(justify right)
+			)
+		)
+		(pin "AUDIO_OUT" output
+			(at 102.87 149.86 0)
+			(effects
+				(font

Commit message: Preliminary layout complete, done on airpane so needs verification.
Parts:
- added H1, H2, H3, H4: MountingHole_Pad, MountingHole:MountingHole_3.2mm_M3_DIN965_Pad, symbol Mechanical:MountingHole_Pad
Connections:
- new net GND: H1.1, H2.1, H3.1, H4.1

Commit message: Added via stitching.
Parts:
- added FID1, FID2, FID3, FID4, FID5, FID6: Fiducial, Fiducial:Fiducial_1.5mm_Mask3mm, symbol Mechanical:Fiducial

Commit message: Finilizing DRC and ERC
Parts:
- removed FID1, FID2, FID3, FID4, FID5, FID6: Fiducial, Fiducial:Fiducial_1.5mm_Mask3mm, symbol Mechanical:Fiducial
- removed H1, H2, H3, H4: MountingHole_Pad, MountingHole:MountingHole_3.2mm_M3_DIN965_Pad, symbol Mechanical:MountingHole_Pad
Other:
- added sheet Mechanical (mechanical.kicad_sch)
