File: buffer.kicad_sch (KiCad schematic)
At the start: 20 parts, among them J8 SJ-3523-SMT-TR, U3 OPA1622

Commit message: Preliminary layout complete, done on airpane so needs verification.
Parts:
- C32: footprint (none) -> Capacitor_SMD:C_0603_1608Metric
- R25, R26, R27, R28, R49, R50, R51, R52: footprint (none) -> Resistor_SMD:R_0402_1005Metric
Changed lines of the file:
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@@
 			)
 		)
-		(property "Footprint" ""
+		(property "Footprint" "Resistor_SMD:R_0402_1005Metric"
 			(at 70.104 120.904 90)
 			(hide yes)
@@
 			)
 		)
-		(property "Footprint" ""
+		(property "Footprint" "Resistor_SMD:R_0402_1005Metric"
 			(at 147.574 145.796 90)
 			(hide yes)
@@
 			)
 		)
-		(property "Footprint" ""
+		(property "Footprint" "Resistor_SMD:R_0402_1005Metric"
 			(at 108.204 133.604 90)
 			(hide yes)
@@
 			)
 		)
-		(property "Footprint" ""
+		(property "Footprint" "Resistor_SMD:R_0402_1005Metric"
 			(at 133.604 123.444 90)
 			(hide yes)
@@
 			)
 		)
-		(property "Footprint" ""
+		(property "Footprint" "Resistor_SMD:R_0402_1005Metric"
 			(at 136.144 76.454 90)
 			(hide yes)
@@
 			)
 		)
-		(property "Footprint" ""
+		(property "Footprint" "Resistor_SMD:R_0402_1005Metric"
 			(at 101.854 87.884 90)
 			(hide yes)
@@
 			)
 		)
-		(property "Footprint" ""
+		(property "Footprint" "Resistor_SMD:R_0402_1005Metric"
 			(at 147.574 98.806 90)
 			(hide yes)
@@
 			)
 		)
-		(property "Footprint" ""
+		(property "Footprint" "Resistor_SMD:R_0402_1005Metric"
 			(at 71.374 73.914 90)
 			(hide yes)
@@
 			)
 		)
-		(property "Footprint" ""
+		(property "Footprint" "Capacitor_SMD:C_0603_1608Metric"
 			(at 109.5248 52.07 0)
 			(hide yes)

Commit message: Added via stitching.
Parts:
- J8: footprint Connector_Audio:Jack_3.5mm_CUI_SJ-3523-SMT_Horizontal -> connectors:Jack_3.5mm_CUI_SJ-3523-SMT_Horizontal
Changed lines of the file:
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@@
 			)
 		)
-		(property "Footprint" "Connector_Audio:Jack_3.5mm_CUI_SJ-3523-SMT_Horizontal"
+		(property "Footprint" "connectors:Jack_3.5mm_CUI_SJ-3523-SMT_Horizontal"
 			(at 247.65 104.14 0)
 			(hide yes)

Commit message: Picked off the board parts and ordered on DigiKey -- also added notes on schematic.
Parts:
- C18, C19: footprint cap_polymer:WCAP-PSLP_6.3X5.8_DXL_ -> polymers:WCAP-PSLP_6.3X5.8_DXL_
- U3: footprint Package_SON:Texas_S-PVSON-N10 -> integrated_circuits:Texas_S-PVSON-N10
Changed lines of the file:
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@@
 			)
 		)
-		(property "Footprint" "Package_SON:Texas_S-PVSON-N10"
+		(property "Footprint" "integrated_circuits:Texas_S-PVSON-N10"
 			(at 97.79 134.62 0)
 			(hide yes)
@@
 			)
 		)
-		(property "Footprint" "Package_SON:Texas_S-PVSON-N10"
+		(property "Footprint" "integrated_circuits:Texas_S-PVSON-N10"
 			(at 97.79 87.63 0)
 			(hide yes)
@@
 			)
 		)
-		(property "Footprint" "Package_SON:Texas_S-PVSON-N10"
+		(property "Footprint" "integrated_circuits:Texas_S-PVSON-N10"
 			(at 97.79 134.62 0)
 			(hide yes)
@@
 			)
 		)
-		(property "Footprint" "cap_polymer:WCAP-PSLP_6.3X5.8_DXL_"
+		(property "Footprint" "polymers:WCAP-PSLP_6.3X5.8_DXL_"
 			(at 173.99 77.47 0)
 			(hide yes)
@@
 			)
 		)
-		(property "Footprint" "cap_polymer:WCAP-PSLP_6.3X5.8_DXL_"
+		(property "Footprint" "polymers:WCAP-PSLP_6.3X5.8_DXL_"
 			(at 173.99 124.46 0)
 			(hide yes)

Commit message: Finally updated all parts in InvenTree and linked them with KiCAD. Ready for BOM exports to JLC.
Parts:
- C17: symbol #inventree_kicad:C_0U1_X7R_16V_0402 -> inventree_kicad:C_0U1_X7R_25V_0402; IPN 301-0003 -> 301-0018; InvenTree 16 -> 52; Part URL http://10.0.0.33/web/part/16/ -> http://10.0.0.33/web/part/52/
- C32: symbol Device:C -> inventree_kicad:C_2U2_X7R_25V_0603; IPN (none) -> 301-0014; InvenTree (none) -> 48; Part URL (none) -> http://10.0.0.33/web/part/48/
- J8: symbol Connector_Audio:AudioJack3 -> inventree_kicad:AUDIO_JACK_3.5MM_SJ-3523-SMT; IPN (none) -> 310-0007; InvenTree (none) -> 39; Part URL (none) -> http://10.0.0.33/web/part/39/
- R25, R26, R27, R28, R49, R50, R51, R52: symbol Device:R_US -> inventree_kicad:R_0R_0402_0W0625; IPN (none) -> 302-0021; InvenTree (none) -> 57; Part URL (none) -> http://10.0.0.33/web/part/57/
- U3: symbol Amplifier_Audio:OPA1622 -> inventree_kicad:AUDIO_AMP_OPA1622_10SON; IPN (none) -> 307-0004; InvenTree (none) -> 61; Part URL (none) -> http://10.0.0.33/web/part/61/
