File: rail_splitter.kicad_sch (KiCad schematic)
At the start: 3 parts, among them U4 TLE2426xD

Commit message: First rough draft of schematics complete -- missing a lot of PLM/Inventree work. Ran through several Claude reviews.
Connections:
- net V_{OUT} renamed V_{MID}
Changed lines of the file:
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@@
 		)
 	)
-	(hierarchical_label "V_{OUT}"
+	(hierarchical_label "V_{MID}"
 		(shape output)
 		(at 179.07 90.17 0)

Commit message: Preliminary layout complete, done on airpane so needs verification.
Parts:
- C15, C16: footprint (none) -> Capacitor_SMD:C_0603_1608Metric
Changed lines of the file:
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@@
 			)
 		)
-		(property "Footprint" ""
+		(property "Footprint" "Capacitor_SMD:C_0603_1608Metric"
 			(at 169.2148 95.25 0)
 			(hide yes)
@@
 			)
 		)
-		(property "Footprint" ""
+		(property "Footprint" "Capacitor_SMD:C_0603_1608Metric"
 			(at 127.3048 97.79 0)
 			(hide yes)

Commit message: Finally updated all parts in InvenTree and linked them with KiCAD. Ready for BOM exports to JLC.
Parts:
- C15: symbol Device:C -> inventree_kicad:C_1U_X7R_25V_0603; IPN (none) -> 301-0013; InvenTree (none) -> 47; Part URL (none) -> http://10.0.0.33/web/part/47/
- C16: symbol Device:C -> inventree_kicad:C_2U2_X7R_25V_0603; IPN (none) -> 301-0014; InvenTree (none) -> 48; Part URL (none) -> http://10.0.0.33/web/part/48/
- U4: value TLE2426xD -> TLE2426; symbol Reference_Voltage:TLE2426xD -> inventree_kicad:TLE2426QDRG4Q1; IPN (none) -> 307-0005; InvenTree (none) -> 62; Part URL (none) -> http://10.0.0.33/web/part/62/
Changed lines of the file:
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@@
 	)
 	(symbol
-		(lib_id "Reference_Voltage:TLE2426xD")
+		(lib_id "inventree_kicad:TLE2426QDRG4Q1")
 		(at 149.86 95.25 0)
 		(unit 1)
@@
 			)
 		)
-		(property "Value" "TLE2426xD"
+		(property "Value" "TLE2426"
 			(at 149.86 85.09 0)
 			(show_name no)
@@
 			)
 		)
-		(property "Datasheet" "http://www.ti.com/lit/ds/symlink/tle2426.pdf"
+		(property "Datasheet" ""
 			(at 114.3 71.12 0)
 			(hide yes)
@@
 			)
 		)
-		(property "Description" "Precision virtual ground, noise reduction pin, 4V to 40V input, SOIC-8"
+		(property "Description" "Rail Splitter, Precision Virtual Ground 4V-40V 20mA 8-SOIC, AEC-Q100"
+			(at 149.86 95.25 0)
+			(hide yes)
+			(show_name no)
+			(do_not_autoplace no)
+			(effects
+				(font
+					(size 1.27 1.27)
+				)
+			)
+		)
+		(property "InvenTree" "62"
+			(at 149.86 95.25 0)
+			(hide yes)
+			(show_name no)
+			(do_not_autoplace no)
+			(effects
+				(font
+					(size 1.27 1.27)
+				)
+			)
+		)
+		(property "Part URL" "http://10.0.0.33/web/part/62/"
+			(at 149.86 95.25 0)
+			(hide yes)
+			(show_name no)
+			(do_not_autoplace no)
+			(effects
+				(font
+					(size 1.27 1.27)
+				)
+			)
+		)
+		(property "IPN" "307-0005"
 			(at 149.86 95.25 0)
 			(hide yes)
@@
 	)
 	(symbol
-		(lib_id "Device:C")
+		(lib_id "inventree_kicad:C_2U2_X7R_25V_0603")
 		(at 170.18 99.06 180)
 		(unit 1)
@@
 			)
 		)
-		(property "Description" "Unpolarized capacitor"
+		(property "Description" "2.2 µF ±10% 25V Ceramic Capacitor X7R 0603 (1608 Metric)"
+			(at 170.18 99.06 0)
+			(hide yes)
+			(show_name no)
+			(do_not_autoplace no)
+			(effects
+				(font
+					(size 1.27 1.27)
+				)
+			)
+		)
+		(property "InvenTree" "48"
+			(at 170.18 99.06 0)
+			(hide yes)
+			(show_name no)
+			(do_not_autoplace no)
+			(effects
+				(font
+					(size 1.27 1.27)
+				)
+			)
+		)
+		(property "Part URL" "http://10.0.0.33/web/part/48/"
+			(at 170.18 99.06 0)
+			(hide yes)
+			(show_name no)
+			(do_not_autoplace no)
+			(effects
+				(font
+					(size 1.27 1.27)
+				)
+			)
+		)
+		(property "IPN" "301-0014"
 			(at 170.18 99.06 0)
 			(hide yes)
@@
 	)
 	(symbol
-		(lib_id "Device:C")
+		(lib_id "inventree_kicad:C_1U_X7R_25V_0603")
 		(at 128.27 101.6 180)
 		(unit 1)
@@
 			)
 		)
-		(property "Description" "Unpolarized capacitor"
+		(property "Description" "1 µF ±10% 25V Ceramic Capacitor X7R 0603 (1608 Metric)"
 			(at 128.27 101.6 0)
 			(hide yes)
+			(show_name no)
+			(do_not_autoplace no)
+			(effects
+				(font
+					(size 1.27 1.27)
+				)
+			)
+		)
+		(property "InvenTree" "47"
+			(at 128.27 101.6 0)
+			(hide yes)
+			(show_name no)
+			(do_not_autoplace no)
+			(effects
+				(font
+					(size 1.27 1.27)
+				)
+			)
+		)
+		(property "Part URL" "http://10.0.0.33/web/part/47/"
+			(at 128.27 101.6 0)
+			(hide yes)
+			(show_name no)
+			(do_not_autoplace no)
+			(effects
+				(font
+					(size 1.27 1.27)
+				)
+			)
+		)
+		(property "IPN" "301-0013"
+			(at 128.27 101.6 0)
+			(hide yes)
