File: headphone_amp.kicad_pcb (KiCad board)
At the start: 4 copper layers, 60 x 60 mm, 134 parts, among them J1 USB4085-GF-A, J10 MJ-3523-SMT-TR, J2 JST PH2, J3 JST GH2, J4 JST SH3, J5 Header_2x1, J6 JST SH3, J7 415-47-208-41-004000, J8 SJ-3523-SMT-TR, Q1 BSS138, SW1 JST SH2, U1 BQ24074RGTR, U2 OPA1678, U3 OPA1622, U4 TLE2426, U5 TPS61379QWRTERQ1, U6 CD74HC4060, U7 74HC14, U8 74HC02, U9 TLV7A0325

Commit message: Cleaning up DRC after updating symbols to match inventree.
Connections:
- U7 pad 15: (no net) -> GND
- U7 pad 7: unconnected-(U7G-GND-Pad7) -> GND
Changed lines of the file:
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@@
 			)
 		)
-		(property "Description" "0.1 µF ±10% 16V Ceramic Capacitor X7R 0402 (1005 Metric)"
+		(property "Description" "0.1 µF ±10% 25V Ceramic Capacitor X7R 0402 (1005 Metric)"
 			(at 0 0 90)
 			(unlocked yes)
@@
 			)
 		)
-		(property "IPN" "301-0003"
+		(property "IPN" "301-0018"
 			(at 0 0 90)
 			(unlocked yes)
@@
 			)
 		)
-		(property "InvenTree" "16"
+		(property "InvenTree" "52"
 			(at 0 0 90)
 			(unlocked yes)
@@
 			)
 		)
-		(property "Part URL" "http://10.0.0.33/web/part/16/"
+		(property "Part URL" "http://10.0.0.33/web/part/52/"
 			(at 0 0 90)
 			(unlocked yes)
@@
 			(unit
 				(name "G")
-				(pins "14" "7")
+				(pins "7" "14" "15")
 			)
 		)
@@
 			(size 0.254 0.8128)
 			(layers "F.Cu" "F.Mask" "F.Paste")
-			(net "unconnected-(U7G-GND-Pad7)")
+			(net "GND")
 			(pinfunction "GND_7")
 			(pintype "power_in")
@@
 			(size 1.143 1.651)
 			(layers "F.Cu" "F.Mask" "F.Paste")
+			(net "GND")
+			(pinfunction "GND_15")
+			(pintype "power_in")
 		)
 		(embedded_fonts no)
@@
 			)
 		)
-		(property "Description" "0.1 µF ±10% 16V Ceramic Capacitor X7R 0402 (1005 Metric)"
+		(property "Description" "0.1 µF ±10% 25V Ceramic Capacitor X7R 0402 (1005 Metric)"
 			(at 0 0 180)
 			(unlocked yes)
@@
 			)
 		)
-		(property "IPN" "301-0003"
+		(property "IPN" "301-0018"
 			(at 0 0 180)
 			(unlocked yes)
@@
 			)
 		)
-		(property "InvenTree" "16"
+		(property "InvenTree" "52"
 			(at 0 0 180)
 			(unlocked yes)
@@
 			)
 		)
-		(property "Part URL" "http://10.0.0.33/web/part/16/"
+		(property "Part URL" "http://10.0.0.33/web/part/52/"
 			(at 0 0 180)
 			(unlocked yes)
