File: watchdog.kicad_sch (KiCad schematic)
At the start: 25 parts, among them U6 CD74HC4060, U7 74HC14BQ,115, U8 74HC02, U9 TLV7A0325PDBVR

Commit message: Added via stitching.
Parts:
- U7: footprint Package_DFN_QFN:DHVQFN-14-1EP_2.5x3mm_P0.5mm_EP1x1.5mm -> integrated_circuits:DHVQFN14_SOT762-1_NEX
- U9: symbol Regulator_Linear:TPS7A0508PDBV -> integrated_circuits:PWR_LDO_2V5_TLV7A0325PDBVR
Changed lines of the file:
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@@
 			)
 		)
-		(property "Footprint" "Package_DFN_QFN:DHVQFN-14-1EP_2.5x3mm_P0.5mm_EP1x1.5mm"
+		(property "Footprint" "integrated_circuits:DHVQFN14_SOT762-1_NEX"
 			(at 138.43 68.58 0)
 			(hide yes)
@@
 			)
 		)
-		(property "Footprint" "Package_DFN_QFN:DHVQFN-14-1EP_2.5x3mm_P0.5mm_EP1x1.5mm"
+		(property "Footprint" "integrated_circuits:DHVQFN14_SOT762-1_NEX"
 			(at 81.28 29.21 0)
 			(hide yes)
@@
 			)
 		)
-		(property "Footprint" "Package_DFN_QFN:DHVQFN-14-1EP_2.5x3mm_P0.5mm_EP1x1.5mm"
+		(property "Footprint" "integrated_circuits:DHVQFN14_SOT762-1_NEX"
 			(at 260.35 128.27 0)
 			(hide yes)
@@
 	)
 	(symbol
-		(lib_id "Regulator_Linear:TPS7A0508PDBV")
+		(lib_id "integrated_circuits:PWR_LDO_2V5_TLV7A0325PDBVR")
 		(at 181.61 31.75 0)
 		(unit 1)
@@
 			)
 		)
-		(property "Footprint" "Package_DFN_QFN:DHVQFN-14-1EP_2.5x3mm_P0.5mm_EP1x1.5mm"
+		(property "Footprint" "integrated_circuits:DHVQFN14_SOT762-1_NEX"
 			(at 260.35 143.51 0)
 			(hide yes)
@@
 			)
 		)
-		(property "Footprint" "Package_DFN_QFN:DHVQFN-14-1EP_2.5x3mm_P0.5mm_EP1x1.5mm"
+		(property "Footprint" "integrated_circuits:DHVQFN14_SOT762-1_NEX"
 			(at 260.35 113.03 0)
 			(hide yes)
@@
 			)
 		)
-		(property "Footprint" "Package_DFN_QFN:DHVQFN-14-1EP_2.5x3mm_P0.5mm_EP1x1.5mm"
+		(property "Footprint" "integrated_circuits:DHVQFN14_SOT762-1_NEX"
 			(at 212.09 35.56 0)
 			(hide yes)
@@
 			)
 		)
-		(property "Footprint" "Package_DFN_QFN:DHVQFN-14-1EP_2.5x3mm_P0.5mm_EP1x1.5mm"
+		(property "Footprint" "integrated_circuits:DHVQFN14_SOT762-1_NEX"
 			(at 260.35 97.79 0)
 			(hide yes)

Commit message: Picked off the board parts and ordered on DigiKey -- also added notes on schematic.
Parts:
- R36: footprint (none) -> Resistor_SMD:R_0402_1005Metric
Changed lines of the file:
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@@
 			)
 		)
-		(property "Footprint" ""
+		(property "Footprint" "Resistor_SMD:R_0402_1005Metric"
 			(at 41.656 148.336 90)
 			(hide yes)

Commit message: Finally updated all parts in InvenTree and linked them with KiCAD. Ready for BOM exports to JLC.
Parts:
- removed U9: TLV7A0325PDBVR, Package_TO_SOT_SMD:SOT-23-5, symbol integrated_circuits:PWR_LDO_2V5_TLV7A0325PDBVR
- added U9: TLV7A0325, Package_TO_SOT_SMD:SOT-23-5, symbol inventree_kicad:TLV7A0325PDBVR
- C20: symbol Device:C -> inventree_kicad:C_1U_X7R_25V_0603; IPN (none) -> 301-0013; InvenTree (none) -> 47; Part URL (none) -> http://10.0.0.33/web/part/47/
- C21: symbol Device:C -> inventree_kicad:C_0U22_X7R_16V_0402; IPN (none) -> 301-0015; InvenTree (none) -> 49; Part URL (none) -> http://10.0.0.33/web/part/49/
- C22: symbol Device:C -> inventree_kicad:C_4U7_X6S_25V_0603; IPN (none) -> 301-0012; InvenTree (none) -> 46; Part URL (none) -> http://10.0.0.33/web/part/46/
- C23: symbol Device:C -> inventree_kicad:C_0U68_X7S_10V_0402; IPN (none) -> 301-0016; InvenTree (none) -> 50; Part URL (none) -> http://10.0.0.33/web/part/50/
- C27, C28: symbol Device:C -> inventree_kicad:C_2U2_X7R_25V_0603; IPN (none) -> 301-0014; InvenTree (none) -> 48; Part URL (none) -> http://10.0.0.33/web/part/48/
- D4: value 1N4148W-7-F -> 1N4148W; symbol Device:D -> inventree_kicad:D_SWITCHING_100V_300MA_SOD123; IPN (none) -> 308-0002; InvenTree (none) -> 37; Part URL (none) -> http://10.0.0.33/web/part/37/
- R36: symbol Device:R_US -> inventree_kicad:R_220K_0402_1PCT_0W0625; IPN (none) -> 302-0019; InvenTree (none) -> 55; Part URL (none) -> http://10.0.0.33/web/part/55/
- R37: symbol Device:R_US -> inventree_kicad:R_100K_0402_1PCT_0W0625; IPN (none) -> 302-0008; InvenTree (none) -> 23; Part URL (none) -> http://10.0.0.33/web/part/23/
- U6: symbol 74xx:74HC4060 -> inventree_kicad:CD74HC4060PWR; IPN (none) -> 307-0006; InvenTree (none) -> 63; Part URL (none) -> http://10.0.0.33/web/part/63/
- U7: value 74HC14BQ,115 -> 74HC14; symbol 74xx:74HC14 -> inventree_kicad:74HC14BQ,115; IPN (none) -> 307-0007; InvenTree (none) -> 64; Part URL (none) -> http://10.0.0.33/web/part/64/
- U8: symbol 74xx:74HC02 -> inventree_kicad:SN74HC02PWR; IPN (none) -> 307-0008; InvenTree (none) -> 65; Part URL (none) -> http://10.0.0.33/web/part/65/
Connections:
- net GND: now also U9.2 (GND); no longer U7.15 (EPAD), U7.7 (GND)
- net V_{LOGIC}: now also U9.5 (OUT)
- net V_{SYS}: now also U9.1 (IN), U9.3 (EN)

Commit message: Cleaning up DRC after updating symbols to match inventree.
Parts:
- U7: symbol inventree_kicad:74HC14BQ,115 -> #inventree_kicad:74HC14BQ,115
Connections:
- net GND: now also U7.15 (GND), U7.7 (GND)
Changed lines of the file:
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@@
 	)
 	(symbol
+		(lib_name "74HC14BQ,115_2")
 		(lib_id "inventree_kicad:74HC14BQ,115")
 		(at 138.43 68.58 0)
@@
 		(dnp no)
 		(property "Reference" "U7"
-			(at 134.62 62.992 0)
+			(at 140.208 59.69 0)
 			(show_name no)
 			(do_not_autoplace no)
@@
 		)
 		(property "Value" "74HC14"
-			(at 131.318 74.93 0)
+			(at 140.97 77.978 0)
 			(show_name no)
 			(do_not_autoplace no)
@@
 		(pin "14"
 		)
+		(pin "15"
+		)
 		(instances
 			(project "headphone_amp"
@@
 	)
 	(symbol
+		(lib_name "74HC14BQ,115_1")
 		(lib_id "inventree_kicad:74HC14BQ,115")
 		(at 81.28 29.21 0)
@@
 		(dnp no)
 		(property "Reference" "U7"
-			(at 77.724 22.86 0)
+			(at 83.058 20.32 0)
 			(show_name no)
 			(do_not_autoplace no)
@@
 		)
 		(property "Value" "74HC14"
-			(at 75.184 35.814 0)
+			(at 83.82 38.608 0)
 			(show_name no)
 			(do_not_autoplace no)
@@
 		(pin "14"
 		)
+		(pin "15"
+		)
 		(instances
 			(project "headphone_amp"
@@
 	)
 	(symbol
+		(lib_name "74HC14BQ,115_5")
 		(lib_id "inventree_kicad:74HC14BQ,115")
 		(at 260.35 128.27 0)
@@
 		(pin "14"
 		)
+		(pin "15"
+		)
 		(instances
 			(project "headphone_amp"
@@
 	)
 	(symbol
+		(lib_name "74HC14BQ,115_6")
 		(lib_id "inventree_kicad:74HC14BQ,115")
 		(at 260.35 143.51 0)
@@
 		(pin "14"
 		)
+		(pin "15"
+		)
 		(instances
 			(project "headphone_amp"
@@
 	)
 	(symbol
+		(lib_name "74HC14BQ,115_4")
 		(lib_id "inventree_kicad:74HC14BQ,115")
 		(at 260.35 113.03 0)
@@
 		(pin "14"
 		)
+		(pin "15"
+		)
 		(instances
 			(project "headphone_amp"
@@
 	)
 	(symbol
-		(lib_id "inventree_kicad:74HC14BQ,115")
+		(lib_id "#inventree_kicad:74HC14BQ,115")
 		(at 212.09 35.56 0)
 		(unit 7)
@@
 		(pin "14"
 		)
+		(pin "15"
+		)
 		(instances
 			(project "headphone_amp"
@@
 	)
 	(symbol
+		(lib_name "74HC14BQ,115_3")
 		(lib_id "inventree_kicad:74HC14BQ,115")
 		(at 260.35 97.79 0)
@@
 		(pin "14"
 		)
+		(pin "15"
+		)
 		(instances
